File: batteryprotector/batteryprotector.kicad_pcb (KiCad board)
At the start: 2 copper layers, 39 parts, among them J1 AVR-ISP-6, J2 Conn_01x02_Female, Q1 SQJ457EP, Q2 BSS123, Q3 PSMN5R2-60YL, SW1 SW_Push, SW2 SW_Push, U1 MCP1799, U2 ATtiny85-20SU

Commit message: layout start
Parts:
- BT1, J2: moved to B.Cu
- Q1: footprint Package_SO:Vishay_PowerPAK_1212-8_Single -> Package_TO_SOT_SMD:LFPAK56
- moved H1 130.3 mm to (13.6, 56.1)
- moved H2 114.1 mm to (13.9, 81.4)
- moved FID1 77.6 mm to (102.1, 97.6), turned to 90 degrees
- moved SW1 74.8 mm to (99.1, 84.1), turned to 270 degrees
- moved FID2 72.6 mm to (105.7, 97.6), turned to 90 degrees
- moved H4 71.7 mm to (69.8, 57.6)
- moved U2 67.9 mm to (112.6, 86.8), turned to 180 degrees
- moved FID3 67.6 mm to (109.2, 97.6), turned to 90 degrees
- moved H3 58.4 mm to (70.0, 82.7)
- moved SW2 56.3 mm to (119.6, 86.9), turned to 270 degrees
- moved R3 56.1 mm to (99.1, 79.9)
- moved D1 54.2 mm to (99.1, 77.0)
- moved C5 49.9 mm to (102.6, 79.9)
- moved R8 48.5 mm to (108.3, 76.2)
- moved R4 46.9 mm to (105.4, 77.0), turned to 270 degrees
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Other:
- board outline added: 70 x 40 mm

Commit message: routing
Parts:
- removed H1, H2, H3, H4: MountingHole, MountingHole:MountingHole_3.2mm_M3_DIN965
- added R7: 33k, Resistor_SMD:R_0805_2012Metric, F.Cu at (111.1, 76.2)
- J1: value AVR-ISP-6 -> AVR-ISP-10; footprint Connector_PinHeader_2.54mm:PinHeader_2x03_P2.54mm_Vertical -> Connector:Tag-Connect_TC2050-IDC-NL_2x05_P1.27mm_Vertical; moved to B.Cu
- moved FID2 32.2 mm to (130.0, 76.5)
- moved Q1 23.6 mm to (99.6, 87.9), turned to 90 degrees
- moved C6 22.6 mm to (125.0, 78.2), turned to 0 degrees
- moved D3 22.5 mm to (126.5, 87.1), turned to 90 degrees
- moved C3 21.8 mm to (138.4, 80.5), turned to 0 degrees
- moved FID3 21.4 mm to (104.4, 76.7)
- moved U1 19.3 mm to (138.4, 83.3), turned to 270 degrees
- moved C1 17.4 mm to (135.4, 83.3), turned to 90 degrees
- moved FID1 17.1 mm to (117.3, 89.7)
- moved R2 16.1 mm to (136.0, 90.9)
- moved C2 14.2 mm to (122.4, 86.7), turned to 90 degrees
- moved C4 13.4 mm to (139.4, 87.1), turned to 90 degrees
- moved C5 10.9 mm to (104.1, 90.7)
- moved R5 10.5 mm to (137.4, 87.1), turned to 90 degrees
- moved R3 9.91 mm to (104.1, 88.4)
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Connections:
- J1 pad 1: /MISO -> /LED_IN
- J1 pad 3: /SCK -> Net-(J1-Pad3)
- J1 pad 4: /LED_IN -> GND
Routing:
- net +5V: track 0.00 -> 64.1 mm, vias 0 -> 3
- net VBUS: track 0.00 -> 43.2 mm, vias 0 -> 10
- net /V_SENSE: track 0.00 -> 34.3 mm
- net Net-(D1-Pad2): track 0.00 -> 17.8 mm, vias 0 -> 2
- net Net-(R4-Pad2): track 0.00 -> 13.3 mm
- net /LED_IN: track 0.00 -> 11.6 mm, vias 0 -> 1
- net /SCK: track 0.00 -> 10.9 mm, vias 0 -> 1
- net Net-(C5-Pad1): track 0.00 -> 10.5 mm
- net /POWER_GATE: track 0.00 -> 9.96 mm
- net Net-(D4-Pad1): track 0.00 -> 7.40 mm
- net /~RESET: track 0.00 -> 7.02 mm, vias 0 -> 1
- net GND: track 0.00 -> 7.01 mm, vias 0 -> 29
- net Net-(Q2-Pad3): track 0.00 -> 5.51 mm
- net Net-(D1-Pad1): track 0.00 -> 5.09 mm
- net /MISO: track 0.00 -> 3.74 mm, vias 0 -> 1
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- added copper zone on B.Cu, net GND
- added copper zone on F.Cu, net GND
- added copper zone on F.Cu, net Net-(BT1-Pad1)
- added copper zone on F.Cu, net Net-(BT1-Pad2)
- added copper zone on F.Cu, net Net-(D1-Pad2)
Other:
- board size 70 x 40 mm -> 58 x 17 mm
