File: batteryprotector/batteryprotector.sch (KiCad schematic (older format))
At the start: 39 parts, among them J1 AVR-ISP-6, J2 Conn_01x02_Female, Q1 SQJ457EP, Q2 BSS123, Q3 PSMN5R2-60YL, SW1 SW_Push, SW2 SW_Push, U1 MCP1799, U2 ATtiny85-20SU

Commit message: layout start
Parts:
- Q1: footprint Package_SO:Vishay_PowerPAK_1212-8_Single -> Package_TO_SOT_SMD:LFPAK56
Changed lines of the file:
@@
 F 0 "Q1" V 4692 1050 50  0000 C CNN
 F 1 "SQJ457EP" V 4601 1050 50  0000 C CNN
-F 2 "Package_SO:Vishay_PowerPAK_1212-8_Single" H 4550 975 50  0001 L CIN
+F 2 "Package_TO_SOT_SMD:LFPAK56" H 4550 975 50  0001 L CIN
 F 3 "https://www.vishay.com/docs/63684/sis415dnt.pdf" V 4350 1050 50  0001 L CNN
 	1    4350 1050
@@
 	5450 1050 5300 1050
 $Comp
-L power:GND #PWR?
+L power:GND #PWR0121
 U 1 1 60732E45
 P 5300 1200
-F 0 "#PWR?" H 5300 950 50  0001 C CNN
+F 0 "#PWR0121" H 5300 950 50  0001 C CNN
 F 1 "GND" H 5305 1027 50  0000 C CNN
 F 2 "" H 5300 1200 50  0001 C CNN

Commit message: routing
Parts:
- removed H1, H2, H3, H4: MountingHole, MountingHole:MountingHole_3.2mm_M3_DIN965, symbol Mechanical:MountingHole
- removed J1: AVR-ISP-6, Connector_PinHeader_2.54mm:PinHeader_2x03_P2.54mm_Vertical, symbol Connector:AVR-ISP-6
- added J1: AVR-ISP-10, Connector:Tag-Connect_TC2050-IDC-NL_2x05_P1.27mm_Vertical, symbol Connector:AVR-ISP-10
- added R7: 33k, Resistor_SMD:R_0805_2012Metric, symbol Device:R
Connections:
- net +5V: now also J1.2 (VCC), R7.2
- net GND: now also J1.10 (GND), J1.4 (GND), J1.6 (GND), J1.8 (GND)
- net LED_IN: now also J1.1 (MOSI)
- net MISO: now also J1.9 (MISO)
- net SCK: now also J1.7 (SCK)
- net ~RESET: now also J1.5 (~RST), R7.1
Changed lines of the file:
@@
-$EndComp
-$Comp
-L Mechanical:MountingHole H1
-U 1 1 6025B2E9
-P 1000 6400
-F 0 "H1" H 1100 6446 50  0000 L CNN
-F 1 "MountingHole" H 1100 6355 50  0000 L CNN
-F 2 "MountingHole:MountingHole_3.2mm_M3_DIN965" H 1000 6400 50  0001 C CNN
-F 3 "~" H 1000 6400 50  0001 C CNN
-	1    1000 6400
-	1    0    0    -1
-$EndComp
-$Comp
-L Mechanical:MountingHole H2
-U 1 1 6025BA60
-P 1000 6600
-F 0 "H2" H 1100 6646 50  0000 L CNN
-F 1 "MountingHole" H 1100 6555 50  0000 L CNN
-F 2 "MountingHole:MountingHole_3.2mm_M3_DIN965" H 1000 6600 50  0001 C CNN
-F 3 "~" H 1000 6600 50  0001 C CNN
-	1    1000 6600
-	1    0    0    -1
-$EndComp
-$Comp
-L Mechanical:MountingHole H3
-U 1 1 6025C1C4
-P 1000 6800
-F 0 "H3" H 1100 6846 50  0000 L CNN
-F 1 "MountingHole" H 1100 6755 50  0000 L CNN
-F 2 "MountingHole:MountingHole_3.2mm_M3_DIN965" H 1000 6800 50  0001 C CNN
-F 3 "~" H 1000 6800 50  0001 C CNN
-	1    1000 6800
-	1    0    0    -1
-$EndComp
-$Comp
-L Mechanical:MountingHole H4
-U 1 1 6025C1CA
-P 1000 7000
-F 0 "H4" H 1100 7046 50  0000 L CNN
-F 1 "MountingHole" H 1100 6955 50  0000 L CNN
-F 2 "MountingHole:MountingHole_3.2mm_M3_DIN965" H 1000 7000 50  0001 C CNN
-F 3 "~" H 1000 7000 50  0001 C CNN
-	1    1000 7000
-	1    0    0    -1
 $EndComp
 $Comp
@@
 Text Label 10100 1250 0    50   ~ 0
 LED_IN
-$Comp
-L Connector:AVR-ISP-6 J1
-U 1 1 607432D6
-P 8900 3400
-F 0 "J1" H 8571 3496 50  0000 R CNN
-F 1 "AVR-ISP-6" H 8571 3405 50  0000 R CNN
-F 2 "Connector_PinHeader_2.54mm:PinHeader_2x03_P2.54mm_Vertical" V 8650 3450 50  0001 C CNN
-F 3 " ~" H 7625 2850 50  0001 C CNN
-	1    8900 3400
-	1    0    0    -1
-$EndComp
 Wire Wire Line
 	10100 1250 9450 1250
@@
 Wire Wire Line
 	5300 1050 5300 1200
+$Comp
+L Device:R R7
+U 1 1 6073B9ED
+P 9850 3200
+F 0 "R7" H 9920 3246 50  0000 L CNN
+F 1 "33k" H 9920 3155 50  0000 L CNN
+F 2 "Resistor_SMD:R_0805_2012Metric" V 9780 3200 50  0001 C CNN
+F 3 "~" H 9850 3200 50  0001 C CNN
+	1    9850 3200
+	1    0    0    1
+$EndComp
+$Comp
+L power:+5V #PWR01
+U 1 1 6073D1A1
+P 9850 3050
+F 0 "#PWR01" H 9850 2900 50  0001 C CNN
+F 1 "+5V" H 9865 3223 50  0000 C CNN
+F 2 "" H 9850 3050 50  0001 C CNN
+F 3 "" H 9850 3050 50  0001 C CNN
+	1    9850 3050
+	1    0    0    -1
+$EndComp
+Wire Wire Line
+	9300 3500 9850 3500
+Wire Wire Line
+	9850 3500 9850 3350
+$Comp
+L Connector:AVR-ISP-10 J1
+U 1 1 60743E13
+P 8900 3400
+F 0 "J1" H 8570 3496 50  0000 R CNN
+F 1 "AVR-ISP-10" H 8570 3405 50  0000 R CNN
+F 2 "Connector:Tag-Connect_TC2050-IDC-NL_2x05_P1.27mm_Vertical" V 8650 3450 50  0001 C CNN
+F 3 " ~" H 7625 2850 50  0001 C CNN
+	1    8900 3400
+	1    0    0    -1
+$EndComp
 $EndSCHEMATC
